File: MSP430_DemoBoard.kicad_pcb (KiCad board)
At the start: 2 copper layers, 63.5 x 62.2 mm, 30 parts, among them J1 VIN, J2 P1.X, J3 P2.X, J4 JTAG-MSP430, J5 P1_2, SW1 SW_Push_Dual, U1 ADP1720ARMZ-3.3-R7, U2 MSP430F2101IRGE

Commit message: Add Toroid and OSH logos
Parts:
- added G***: TOROID, TOROID-KiCad:Logo_and_Name_20mm_FSilk, F.Cu at (163.8, 67.3)
- added REF***: OSHW-Logo2_14.6x12mm_SilkScreen, Symbols:OSHW-Logo2_14.6x12mm_SilkScreen, F.Cu at (151.1, 55.9)

Commit message: Routing
Parts:
- removed the G*** at (163.8, 67.3)
- removed J5: P1_2, Pin_Headers:Pin_Header_Straight_2x08_Pitch2.54mm
- added D4: LED, LEDs:LED_0603, F.Cu at (157.4, 89.8)
- added D5: LED, LEDs:LED_0603, F.Cu at (155.5, 89.8)
- added G***: TOROID, TOROID-KiCad:Logo_and_Name_32mm_FSilk, F.Cu at (169.7, 45.6)
- added R6: 330, Resistors_SMD:R_0603_HandSoldering, F.Cu at (157.4, 85.7)
- added R7: 330, Resistors_SMD:R_0603_HandSoldering, F.Cu at (155.5, 85.7)
- added REF**: ThermalVia_0.3mm, TOROID-KiCad:ThermalVia_0.3mm, F.Cu at (159.0, 69.1)
- added REF**: ThermalVia_0.3mm, TOROID-KiCad:ThermalVia_0.3mm, F.Cu at (158.5, 68.6)
- added REF**: ThermalVia_0.3mm, TOROID-KiCad:ThermalVia_0.3mm, F.Cu at (159.5, 69.6)
- added REF**: ThermalVia_0.3mm, TOROID-KiCad:ThermalVia_0.3mm, F.Cu at (159.0, 68.1)
- added REF**: ThermalVia_0.3mm, TOROID-KiCad:ThermalVia_0.3mm, F.Cu at (159.5, 68.6)
- added REF**: ThermalVia_0.3mm, TOROID-KiCad:ThermalVia_0.3mm, F.Cu at (160.0, 69.1)
- added REF**: ThermalVia_0.3mm, TOROID-KiCad:ThermalVia_0.3mm, F.Cu at (160.5, 68.6)
- added REF**: ThermalVia_0.3mm, TOROID-KiCad:ThermalVia_0.3mm, F.Cu at (160.0, 68.1)
- added REF**: ThermalVia_0.3mm, TOROID-KiCad:ThermalVia_0.3mm, F.Cu at (159.5, 67.6)
- moved JP1 52.9 mm to (189.7, 45.7), turned to 0 degrees
- moved J4 51.3 mm to (167.9, 94.4), turned to 270 degrees
- moved J1 45.8 mm to (197.1, 48.4), turned to 270 degrees
- moved JP3 45.1 mm to (168.9, 84.0), turned to 270 degrees
- moved C2 40.0 mm to (196.7, 51.4), turned to 0 degrees
- moved JP2 36.5 mm to (166.4, 79.5), turned to 90 degrees
- moved U1 33.4 mm to (196.7, 55.2), turned to 0 degrees
- moved RV1 33.0 mm to (175.9, 85.7), turned to 270 degrees
- moved C3 28.3 mm to (196.7, 58.4), turned to 0 degrees
- moved D1 27.6 mm to (163.2, 89.8), turned to 90 degrees
- moved REF*** 26.7 mm to (177.8, 56.6), turned to 0 degrees
- moved C4 25.5 mm to (196.7, 60.3)
- moved D2 23.3 mm to (161.2, 89.8), turned to 90 degrees
- moved R3 21.9 mm to (163.2, 85.7), turned to 270 degrees
- moved R1 20.6 mm to (168.9, 67.9), turned to 180 degrees
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Connections:
- J3 pad 1: /P2.0 -> /P2.5
- J3 pad 2: /P2.1 -> /P2.7
- J3 pad 3: /P2.2 -> /P2.6
- J3 pad 4: /P2.3 -> /P2.0
- J3 pad 5: /P2.4 -> /P2.1
- J3 pad 6: /P2.5 -> /P2.2
- J3 pad 7: /P2.6 -> /P2.3
- J3 pad 8: /P2.7 -> /P2.4
- RV1 pad 1: /VCC -> GND
- RV1 pad 3: GND -> /VCC
- RV2 pad 1: /VCC -> GND
- RV2 pad 3: GND -> /VCC
- RV3 pad 1: /VCC -> GND
- RV3 pad 3: GND -> /VCC
Routing:
- net /VCC: track 0.00 -> 82.2 mm
- net /P1.7: track 0.00 -> 64.3 mm
- net /P2.3: track 0.00 -> 63.4 mm, vias 0 -> 2
- net /P2.4: track 0.00 -> 60.4 mm, vias 0 -> 2
- net /P1.6: track 0.00 -> 59.1 mm, vias 0 -> 1
- net /P2.5: track 0.00 -> 55.5 mm, vias 0 -> 2
- net /RST: track 0.00 -> 55.3 mm, vias 0 -> 3
- net /P1.4: track 0.00 -> 53.3 mm, vias 0 -> 1
- net /P1.5: track 0.00 -> 53.1 mm, vias 0 -> 1
- net /P1.1: track 0.00 -> 42.7 mm, vias 0 -> 1
- net /P1.2: track 0.00 -> 40.4 mm, vias 0 -> 1
- net /P1.3: track 0.00 -> 38.2 mm, vias 0 -> 1
- net /TEST: track 0.00 -> 36.5 mm, vias 0 -> 1
- net /P2.7: track 0.00 -> 27.2 mm
- net GND: track 0.00 -> 26.8 mm, vias 0 -> 3
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- added copper zone on F.Cu, net /VCC
- added copper zone on B.Cu, net GND
- added copper zone on F.Cu, net GND
- added copper zone on F.Cu, net Net-(C2-Pad1)

Commit message: SilkS comments
Other:
- board text added: "+-"
- board text added: "1"
- board text added: "5V"
- board text added: "EN"
- board text added: "JTAG"
- board text added: "P1.0"
- board text added: "P1.1"
- board text added: "P1.2"
- board text added: "P1.3"
- board text added: "P1.4"
- board text added: "P1.5"
- board text added: "P1.6"
- board text added: "P1.7"
- board text added: "P2.0"
- board text added: "P2.1"
- board text added: "P2.2"
- board text added: "P2.3"
- board text added: "P2.4"
- board text added: "P2.5"
- board text added: "P2.6"
- board text added: "P2.7"
- board text added: "TARGET"
- board text added: "TOOL"
- board text added: "VCC"
