File: MSP430_DemoBoard.kicad_pcb (KiCad board)
At the start: 2 copper layers, 63.5 x 62.2 mm, 44 parts, among them J1 VIN, J2 P1.X, J3 P2.X, J4 JTAG-MSP430, SW1 SW_Push_Dual, U1 ADP1720ARMZ-3.3-R7, U2 MSP430F2101IRGE

Commit message: Add commit-trace. Remove signature
Parts:
- added REF**: commit-trace-small, toroid-kicad:commit-trace, F.Cu at (164.0, 55.5)
Changed lines of the file:
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@@
-(kicad_pcb (version 20170123) (host pcbnew "(2017-02-17 revision 0898b6c94)-makepkg")
+(kicad_pcb (version 20170123) (host pcbnew "(2017-05-18 revision 2a3a699d9)-master")
   (general
-    (links 83)
+    (links 0)
     (no_connects 0)
     (area 139.354048 36.9325 206.085953 101.6325)
@@
     (tracks 258)
     (zones 0)
-    (modules 44)
+    (modules 45)
     (nets 31)
   )
@@
     (add_net "Net-(R2-Pad2)")
   )
+  (module toroid-kicad:commit-trace (layer F.Cu)
+    (at 164 55.5)
+    (fp_text reference REF** (at -5.3 3.5) (layer F.SilkS) hide
+      (effects (font (size 1 1) (thickness 0.15)))
+    )
+    (fp_text value commit-trace-small (at 0.1 -4.4) (layer F.Fab) hide
+      (effects (font (size 1 1) (thickness 0.15)))
+    )
+    (fp_text user $date$ (at 3.25 1.5) (layer F.SilkS)
+      (effects (font (size 0.8 0.8) (thickness 0.2)))
+    )
+    (fp_text user $tag$ (at 3.25 -0.25) (layer F.SilkS)
+      (effects (font (size 0.8 0.8) (thickness 0.2)))
+    )
+    (fp_text user $commit$ (at 3.25 -2) (layer F.SilkS)
+      (effects (font (size 0.8 0.8) (thickness 0.2)))
+    )
+    (fp_arc (start 6.75 -2.25) (end 7.5 -2.25) (angle -90) (layer F.SilkS) (width 0.15))
+    (fp_arc (start 6.75 1.75) (end 6.75 2.5) (angle -90) (layer F.SilkS) (width 0.15))
+    (fp_arc (start -6.75 1.75) (end -7.5 1.75) (angle -90) (layer F.SilkS) (width 0.15))
+    (fp_arc (start -6.75 -2.25) (end -6.75 -3) (angle -90) (layer F.SilkS) (width 0.15))
+    (fp_line (start -7.5 1.75) (end -7.5 -2.25) (layer F.SilkS) (width 0.15))
+    (fp_line (start 6.75 2.5) (end -6.75 2.5) (layer F.SilkS) (width 0.15))
+    (fp_line (start 7.5 -2.25) (end 7.5 1.75) (layer F.SilkS) (width 0.15))
+    (fp_line (start -6.75 -3) (end 6.75 -3) (layer F.SilkS) (width 0.15))
+    (fp_text user DATE: (at -5 1.5) (layer F.SilkS)
+      (effects (font (size 1 1) (thickness 0.15) italic))
+    )
+    (fp_text user TAG: (at -5.5 -0.25) (layer F.SilkS)
+      (effects (font (size 1 1) (thickness 0.15) italic))
+    )
+    (fp_text user COMMIT: (at -4 -2) (layer F.SilkS)
+      (effects (font (size 1 1) (thickness 0.15) italic))
+    )
+  )
   (module Symbols:OSHW-Logo2_14.6x12mm_SilkScreen (layer F.Cu)

Commit message: PCB Update
Parts:
- removed JP1: Enable, Pin_Headers:Pin_Header_Straight_1x02_Pitch2.54mm
- moved C2 0.96 mm to (195.8, 51.5)
Connections:
- J4 pad 10: (no net) -> Net-(J4-Pad10)
- J4 pad 12: (no net) -> Net-(J4-Pad12)
- J4 pad 13: (no net) -> Net-(J4-Pad13)
- J4 pad 14: (no net) -> Net-(J4-Pad14)
- J4 pad 6: (no net) -> Net-(J4-Pad6)
- SW1 pad 1: (no net) -> Net-(SW1-Pad1)
- SW1 pad 2: (no net) -> Net-(SW1-Pad2)
- U1 pad 4: Net-(JP1-Pad2) -> Net-(C2-Pad1)
Routing:
- net /VCC: track 82.2 -> 100.9 mm
- net Net-(JP1-Pad2): track 11.3 -> 0.00 mm, vias 1 -> 0
- net GND: track 26.8 -> 28.5 mm
- net Net-(C2-Pad1): track 9.62 -> 11.1 mm
- net /P2.7: track 27.2 -> 27.7 mm
- removed copper zone on F.Cu, net /VCC
- removed copper zone on F.Cu, net Net-(C2-Pad1)
Other:
- board text removed: "EN"
